File: board/board.kicad_sch (KiCad schematic)
At the start: 1 part

Commit message: initial
Parts:
- removed LOGO1: Logo_Open_Hardware_Small, Symbol:OSHW-Symbol_6.7x6mm_SilkScreen, symbol Graphic:Logo_Open_Hardware_Small
- added J1: Conn_Coaxial, Connector_Coaxial:SMA_Molex_73251-1153_EdgeMount_Horizontal, symbol Connector:Conn_Coaxial
- added J2: 007_ADC_2x2, on_edge:on_edge_2x05_device, symbol put_on_edge:007_ADC
- added R1: d.n.p, Resistor_SMD:R_0603_1608Metric, symbol Device:R_Small
Connections:
- new net: J1.1 (In), J2.3 (ADC0)
- new net: J1.2 (Ext), J2.4 (ADC1), R1.1
- new net GND: J2.1 (GND), R1.2
- no-connect marks 0 -> 5
Other:
- removed sheet implementation
- note removed: "Input connectors go here"
- note removed: "Output connectors go here"
Changed lines of the file:
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@@
 (kicad_sch (version 20211123) (generator eeschema)
   (paper "A4")
-  (text "Output connectors go here" (at 224.79 88.9 0)
-    (effects (font (size 1.27 1.27)) (justify left bottom))
+  (junction (at 116.205 97.155) (diameter 0) (color 0 0 0 0)
   )
-  (text "Input connectors go here" (at 49.53 88.9 0)
-    (effects (font (size 1.27 1.27)) (justify left bottom))
+  (no_connect (at 99.06 95.25))
+  (no_connect (at 99.06 102.87))
+  (no_connect (at 99.06 105.41))
+  (no_connect (at 99.06 97.79))
+  (no_connect (at 99.06 87.63))
+  (wire (pts (xy 109.22 97.155) (xy 116.205 97.155))
+    (stroke (width 0) (type default) (color 0 0 0 0))
   )
-  (symbol (lib_id "Graphic:Logo_Open_Hardware_Small") (at 273.05 157.48 0) (unit 1)
-    (in_bom yes) (on_board yes) (fields_autoplaced)
-    (property "Reference" "LOGO1" (id 0) (at 273.05 150.495 0)
+  (wire (pts (xy 87.63 113.03) (xy 87.63 116.205))
+    (stroke (width 0) (type default) (color 0 0 0 0))
+  )
+  (wire (pts (xy 99.06 92.71) (xy 109.22 92.71))
+    (stroke (width 0) (type default) (color 0 0 0 0))
+  )
+  (wire (pts (xy 116.205 97.79) (xy 116.205 97.155))
+    (stroke (width 0) (type default) (color 0 0 0 0))
+  )
+  (wire (pts (xy 99.06 90.17) (xy 111.125 90.17))
+    (stroke (width 0) (type default) (color 0 0 0 0))
+  )
+  (wire (pts (xy 109.22 92.71) (xy 109.22 97.155))
+    (stroke (width 0) (type default) (color 0 0 0 0))
+  )
+  (wire (pts (xy 116.205 107.315) (xy 116.205 102.87))
+    (stroke (width 0) (type default) (color 0 0 0 0))
+  )
+  (wire (pts (xy 116.205 97.155) (xy 116.205 95.25))
+    (stroke (width 0) (type default) (color 0 0 0 0))
+  )
+  (symbol (lib_id "Connector:Conn_Coaxial") (at 116.205 90.17 0) (unit 1)
+    (in_bom yes) (on_board yes)
+    (property "Reference" "J1" (id 0) (at 118.745 90.805 0)
+      (effects (font (size 1.27 1.27)) (justify left))
+    )
+    (property "Value" "Conn_Coaxial" (id 1) (at 118.745 93.1164 0)
+      (effects (font (size 1.27 1.27)) (justify left))
+    )
+    (property "Footprint" "Connector_Coaxial:SMA_Molex_73251-1153_EdgeMount_Horizontal" (id 2) (at 116.205 90.17 0)
       (effects (font (size 1.27 1.27)) hide)
     )
-    (property "Value" "Logo_Open_Hardware_Small" (id 1) (at 273.05 163.195 0)
+    (property "Datasheet" " ~" (id 3) (at 116.205 90.17 0)
       (effects (font (size 1.27 1.27)) hide)
     )
-    (property "Footprint" "Symbol:OSHW-Symbol_6.7x6mm_SilkScreen" (id 2) (at 273.05 157.48 0)
+    (pin "1")
+    (pin "2")
+  )
+  (symbol (lib_id "Device:R_Small") (at 116.205 100.33 0) (unit 1)
+    (in_bom yes) (on_board yes)
+    (property "Reference" "R1" (id 0) (at 117.7036 99.1616 0)
+      (effects (font (size 1.27 1.27)) (justify left))
+    )
+    (property "Value" "d.n.p" (id 1) (at 117.7036 101.473 0)
+      (effects (font (size 1.27 1.27)) (justify left))
+    )
+    (property "Footprint" "Resistor_SMD:R_0603_1608Metric" (id 2) (at 116.205 100.33 0)
       (effects (font (size 1.27 1.27)) hide)
     )
-    (property "Datasheet" "~" (id 3) (at 273.05 157.48 0)
+    (property "Datasheet" "~" (id 3) (at 116.205 100.33 0)
       (effects (font (size 1.27 1.27)) hide)
     )
+    (pin "1")
+    (pin "2")
   )
-  (sheet (at 114.3 72.39) (size 60.96 62.23) (fields_autoplaced)
-    (stroke (width 0.1524) (type solid) (color 0 0 0 0))
-    (fill (color 0 0 0 0.0000))
-    (property "Sheet name" "implementation" (id 0) (at 114.3 71.6784 0)
-      (effects (font (size 1.27 1.27)) (justify left bottom))
+  (symbol (lib_id "power:GND") (at 116.205 107.315 0) (mirror y) (unit 1)
+    (in_bom yes) (on_board yes)
+    (property "Reference" "#PWR0101" (id 0) (at 116.205 113.665 0)
+      (effects (font (size 1.27 1.27)) hide)
     )
-    (property "Sheet file" "implementation.kicad_sch" (id 1) (at 114.3 135.2046 0)
-      (effects (font (size 1.27 1.27)) (justify left top))
+    (property "Value" "GND" (id 1) (at 116.078 111.7092 0))
+    (property "Footprint" "" (id 2) (at 116.205 107.315 0)
+      (effects (font (size 1.27 1.27)) hide)
     )
+    (property "Datasheet" "" (id 3) (at 116.205 107.315 0)
+      (effects (font (size 1.27 1.27)) hide)
+    )
+    (pin "1")
+  )
+  (symbol (lib_id "put_on_edge:007_ADC") (at 87.63 95.25 0) (mirror y) (unit 1)
+    (in_bom yes) (on_board yes)
+    (property "Reference" "J2" (id 0) (at 79.2988 94.9198 0)
+      (effects (font (size 1.27 1.27)) (justify left))
+    )
+    (property "Value" "007_ADC_2x2" (id 1) (at 79.2988 97.2312 0)
+      (effects (font (size 1.27 1.27)) (justify left))
+    )
+    (property "Footprint" "on_edge:on_edge_2x05_device" (id 2) (at 80.01 78.74 0)
+      (effects (font (size 1.27 1.27)) hide)
+    )
+    (property "Datasheet" "" (id 3) (at 80.01 78.74 0)
+      (effects (font (size 1.27 1.27)) hide)
+    )
+    (pin "1")
+    (pin "10")
+    (pin "2")
+    (pin "3")
+    (pin "4")
+    (pin "5")
+    (pin "6")
+    (pin "9")
+  )
+  (symbol (lib_id "power:GND") (at 87.63 116.205 0) (mirror y) (unit 1)
+    (in_bom yes) (on_board yes)
+    (property "Reference" "#PWR0112" (id 0) (at 87.63 122.555 0)
+      (effects (font (size 1.27 1.27)) hide)
+    )
+    (property "Value" "GND" (id 1) (at 87.503 120.5992 0))
+    (property "Footprint" "" (id 2) (at 87.63 116.205 0)
+      (effects (font (size 1.27 1.27)) hide)
+    )
+    (property "Datasheet" "" (id 3) (at 87.63 116.205 0)
+      (effects (font (size 1.27 1.27)) hide)
+    )
+    (pin "1")
   )
   (sheet_instances
     (path "/" (page "1"))
-    (path "/767ce4c6-0e55-4543-92f0-34cb8237a544" (page "2"))
   )
   (symbol_instances
-    (path "/b72b6f4a-7489-40f2-bb90-d75ae01aa368"
-      (reference "LOGO1") (unit 1) (value "Logo_Open_Hardware_Small") (footprint "Symbol:OSHW-Symbol_6.7x6mm_SilkScreen")
+    (path "/00000000-0000-0000-0000-00006034079d"
+      (reference "#PWR0101") (unit 1) (value "GND") (footprint "")
+    )
+    (path "/00000000-0000-0000-0000-00006034e58c"
+      (reference "#PWR0112") (unit 1) (value "GND") (footprint "")
+    )
+    (path "/00000000-0000-0000-0000-00006033f336"
+      (reference "J1") (unit 1) (value "Conn_Coaxial") (footprint "Connector_Coaxial:SMA_Molex_73251-1153_EdgeMount_Horizontal")
+    )
+    (path "/00000000-0000-0000-0000-00006034b92f"
+      (reference "J2") (unit 1) (value "007_ADC_2x2") (footprint "on_edge:on_edge_2x05_device")
+    )
+    (path "/00000000-0000-0000-0000-0000603401d4"
+      (reference "R1") (unit 1) (value "d.n.p") (footprint "Resistor_SMD:R_0603_1608Metric")
     )
   )
